File: Arty_HDMI_SD/HDMI_SD_expansion.sch (KiCad schematic (older format))
At the start: 13 parts, among them J1 0015912120, J2 SD_card_slot, J3 0015912120, J4 HDMI_A

Commit message: Replaced HDMI connector
Parts:
- removed J4: HDMI_A, antmicro-footprints:HDMI_A_Female_2000-1-2-41-00-BK, symbol Connector:HDMI_A
- added J4: 2000-1-2-41-00-BK, antmicro-footprints:HDMI_A_Female_2000-1-2-41-00-BK, symbol antmicro_USB_DVI_HDMI_Connectors:2000-1-2-41-00-BK
Connections:
- wire segments 112 -> 107
Other:
- note added: "HDMI_CON_#2"
- note added: "HDMI_INTERFACE"
- note added: "SD_CARD_SLOT"
- note added: "SD_CON_#1"
- moved on the sheet: J1, J3, R1, R2, R3, R4, R5, R6, R7

Commit message: Review
Other:
- note added: "CK and MOSI doubled\n"
- note added: "Connect all TMDS signals via 100n capacitors.\nWe can always replace them with 0R resistors"
- note added: "VCC is 3V3 in PMOD standard"
- note added: "generally some connections for SD are wrong. \nI suggest using: \nhttps://store.digilentinc.com/pmod-microsd-microsd-card-slot/ \nas reference\n"
- note added: "swapped P with N\n"
- note added: "there is no 5V coming from PMOD, we can leave it floating\n"
- note added: "why TMDS here?\n"
Changed lines of the file:
@@
 Text Notes 1100 4100 0    98   ~ 0
 SD_CARD_SLOT
+Text Notes 3300 1950 0    50   ~ 10
+why TMDS here?\n
+Text Notes 750  2050 0    50   ~ 10
+CK and MOSI doubled\n
+Text Notes 1700 2450 0    50   ~ 10
+VCC is 3V3 in PMOD standard
+Text Notes 6900 2600 0    50   ~ 10
+VCC is 3V3 in PMOD standard
+Text Notes 8750 4300 0    50   ~ 10
+there is no 5V coming from PMOD, we can leave it floating\n
+Text Notes 2800 4500 0    50   ~ 10
+generally some connections for SD are wrong. \nI suggest using: \nhttps://store.digilentinc.com/pmod-microsd-microsd-card-slot/ \nas reference\n
+Text Notes 8350 5000 0    50   ~ 10
+swapped P with N\n
+Text Notes 8450 2350 0    50   ~ 10
+Connect all TMDS signals via 100n capacitors.\nWe can always replace them with 0R resistors
 $EndSCHEMATC

Commit message: Added USB SPI Interface
Parts:
- removed C1: C_1u_0603, antmicro-footprints:0603-cap, symbol antmicro_Capacitors_0603:C_1u_0603
- removed D1: TPD6E05U06, antmicro-footprints:TPD6E05U06, symbol antmicro_TVS_Diodes:TPD6E05U06
- removed J2: SD_card_slot, antmicro-footprints:1140084168, symbol HDMI_SD_expansion-rescue:SD_card_slot-antmicro_Memory_Connectors_PC_Card_Sockets
- removed R1, R2, R3, R4, R5, R6, R7: R_10k_0603, antmicro-footprints:0603-res, symbol antmicro_Resistors_0603:R_10k_0603
- added C1, C15, C18, C19, C2, C3, C4, C5, C6, C7, C8, C9: C_100n_0402_6V3, antmicro-footprints:0402-cap, symbol antmicro_Capacitors_0402:C_100n_0402_6V3
- added C10, C12, C13, C14: C_22u_0603, antmicro-footprints:0603-cap, symbol antmicro_Capacitors_0603:C_22u_0603
- added C11: C_10n_0402, antmicro-footprints:0402-cap, symbol antmicro_Capacitors_0402:C_10n_0402
- added C16, C17: C_22p_0402, antmicro-footprints:0402-cap, symbol antmicro_Capacitors_0402:C_22p_0402
- added D1, D2: PGB1010603MR, antmicro-footprints:0603, symbol antmicro_TVS_Diodes:PGB1010603MR
- added FB1, FB2: BLM21PG221SN1D, antmicro-footprints:0805, symbol antmicro_Ferrite_Beads_and_Chips:BLM21PG221SN1D
- added J2: 1140084168, antmicro-footprints:MicroSD_1140084168, symbol antmicro_Memory_Connectors_PC_Card_Sockets:1140084168
- added J5: UE27AC54100, antmicro-footprints:USB_A_Female_UE27AC54100, symbol antmicro_USB_DVI_HDMI_Connectors:UE27AC54100
- added J6: 0015912120, antmicro-footprints:PinHeader_6x2_P2.54mm_Horizontal_Mirrored, symbol antmicro_Rectangular_Connectors_Headers_Male_Pins:0015912120
- added L1: XFL4020-102MEB, antmicro-footprints:XFL4020-102MEB, symbol antmicro_Fixed_Inductors:XFL4020-102MEB
- added R1, R2, R3, R4, R5, R6, R7: R_20k_0603, antmicro-footprints:0603-res, symbol antmicro_Resistors_0603:R_20k_0603
- added R10, R9: R_22R_0402, antmicro-footprints:0402-res, symbol antmicro_Resistors_0402:R_22R_0402
- added R11, R8: R_0R_0603, antmicro-footprints:0603-res, symbol antmicro_Resistors_0603:R_0R_0603
- added R12: R_220R_0402, antmicro-footprints:0402-res, symbol antmicro_Resistors_0402:R_220R_0402
- added TP1, TP2, TP3: TP_SMD1MM, antmicro-footprints:Testpoint_smd_1mm, symbol antmicro_Test_Points:TP_SMD1MM
- added U1: TPS61232DRCT, antmicro-footprints:VSON-10-1EP_3x3mm, symbol antmicro_DC_DC_Converters:TPS61232DRCT
- added U2: MAX3421EEHJ, antmicro-footprints:TQFP-32_5x5mm, symbol antmicro_Interface_Controllers:MAX3421EEHJ
- added Y1: KX-7_12,MHz, antmicro-footprints:KX-7, symbol antmicro_Oscillators:KX-7_12,MHz
- J1, J3: footprint antmicro-footprints:PinHeader_6x2_P2.54mm_Horizontal -> antmicro-footprints:PinHeader_6x2_P2.54mm_Horizontal_Mirrored
Connections:
- net labels added: CD_DAT3, C_TDMS_CLK_N, C_TDMS_CLK_P, C_TDMS_D0_N, C_TDMS_D0_P, C_TDMS_D1_N, C_TDMS_D1_P, C_TDMS_D2_N, C_TDMS_D2_P, GPX_USB, MISO_DAT0, MISO_USB, MOSI_CMD, MOSI_USB, NC_EN, RST_USB, SCK_USB, SS_USB
- net labels removed: CD1, CD2, MISO, MOSI, SS
- wire segments 107 -> 248
Other:
- note added: "?"
- note added: "Co to jest? Było w tym Reference od \nArduino i w bibliotece to wstawiłem."
- note added: "DC-DC Step UP"
- note added: "Dodać ogranicznik prądu?"
- note added: "Tutaj jeszcze bezpiecznik na 500mA \nale chyba musze go zrobic najpierw"
- note added: "USB_CON_#3"
- note removed: "CK and MOSI doubled\n"
- note removed: "Connect all TMDS signals via 100n capacitors.\nWe can always replace them with 0R resistors"
- note removed: "VCC is 3V3 in PMOD standard"
- note removed: "generally some connections for SD are wrong. \nI suggest using: \nhttps://store.digilentinc.com/pmod-microsd-microsd-card-slot/ \nas reference\n"
- note removed: "swapped P with N\n"
- note removed: "there is no 5V coming from PMOD, we can leave it floating\n"
- note removed: "why TMDS here?\n"
- moved on the sheet: J1, J3, J4

Commit message: Schematic updates
Parts:
- removed FB1: BLM21PG221SN1D, antmicro-footprints:0805, symbol antmicro_Ferrite_Beads_and_Chips:BLM21PG221SN1D
- removed R11: R_0R_0603, antmicro-footprints:0603-res, symbol antmicro_Resistors_0603:R_0R_0603
- added R11: R_10k_0603, antmicro-footprints:0603-res, symbol antmicro_Resistors_0603:R_10k_0603
- C1, C15, C18, C19, C2, C3, C4, C5, C6, C7, C8, C9: symbol antmicro_Capacitors_0402:C_100n_0402_6V3 -> HDMI_SD_expansion-rescue:C_100n_0402_6V3-antmicro_Capacitors_0402
Connections:
- wire segments 248 -> 244
Other:
- note added: "caps will be replaced with 0R by default"
- note removed: "Co to jest? Było w tym Reference od \nArduino i w bibliotece to wstawiłem."
- note removed: "Dodać ogranicznik prądu?"
- note removed: "Tutaj jeszcze bezpiecznik na 500mA \nale chyba musze go zrobic najpierw"
- moved on the sheet: J5
Changed lines of the file:
@@
 	1950 6600 3900 6600
 $Comp
-L antmicro_Capacitors_0402:C_100n_0402_6V3 C2
+L HDMI_SD_expansion-rescue:C_100n_0402_6V3-antmicro_Capacitors_0402 C2
 U 1 1 5D82C2CC
 P 3100 3150
@@
 $EndComp
 $Comp
-L antmicro_Capacitors_0402:C_100n_0402_6V3 C3
+L HDMI_SD_expansion-rescue:C_100n_0402_6V3-antmicro_Capacitors_0402 C3
 U 1 1 5D82C3D2
 P 3350 3150
@@
 $EndComp
 $Comp
-L antmicro_Capacitors_0402:C_100n_0402_6V3 C4
+L HDMI_SD_expansion-rescue:C_100n_0402_6V3-antmicro_Capacitors_0402 C4
 U 1 1 5D82FF3B
 P 3600 3150
@@
 $EndComp
 $Comp
-L antmicro_Capacitors_0402:C_100n_0402_6V3 C5
+L HDMI_SD_expansion-rescue:C_100n_0402_6V3-antmicro_Capacitors_0402 C5
 U 1 1 5D82FF7F
 P 3850 3150
@@
 $EndComp
 $Comp
-L antmicro_Capacitors_0402:C_100n_0402_6V3 C6
+L HDMI_SD_expansion-rescue:C_100n_0402_6V3-antmicro_Capacitors_0402 C6
 U 1 1 5D8300D9
 P 4100 3150
@@
 $EndComp
 $Comp
-L antmicro_Capacitors_0402:C_100n_0402_6V3 C7
+L HDMI_SD_expansion-rescue:C_100n_0402_6V3-antmicro_Capacitors_0402 C7
 U 1 1 5D8300E3
 P 4350 3150
@@
 $EndComp
 $Comp
-L antmicro_Capacitors_0402:C_100n_0402_6V3 C8
+L HDMI_SD_expansion-rescue:C_100n_0402_6V3-antmicro_Capacitors_0402 C8
 U 1 1 5D8300ED
 P 4600 3150
@@
 $EndComp
 $Comp
-L antmicro_Capacitors_0402:C_100n_0402_6V3 C9
+L HDMI_SD_expansion-rescue:C_100n_0402_6V3-antmicro_Capacitors_0402 C9
 U 1 1 5D8300F7
 P 4850 3150
@@
 $EndComp
 $Comp
-L antmicro_Capacitors_0402:C_100n_0402_6V3 C1
+L HDMI_SD_expansion-rescue:C_100n_0402_6V3-antmicro_Capacitors_0402 C1
 U 1 1 5D7BA763
 P 3350 7050
@@
 Connection ~ 3350 5200
 $Comp
-L antmicro_Capacitors_0402:C_100n_0402_6V3 C18
+L HDMI_SD_expansion-rescue:C_100n_0402_6V3-antmicro_Capacitors_0402 C18
 U 1 1 5D7247BC
 P 8250 5950
@@
 	9650 3850 9650 4050
 $Comp
-L antmicro_Capacitors_0402:C_100n_0402_6V3 C19
+L HDMI_SD_expansion-rescue:C_100n_0402_6V3-antmicro_Capacitors_0402 C19
 U 1 1 5D77BBF9
 P 10250 3850
@@
 L antmicro_USB_DVI_HDMI_Connectors:UE27AC54100 J5
 U 1 1 5D7BA5ED
-P 6000 4550
-F 0 "J5" H 5900 4850 60  0000 C CNN
-F 1 "UE27AC54100" H 5800 4200 60  0000 C CNN
-F 2 "antmicro-footprints:USB_A_Female_UE27AC54100" H 6200 4750 60  0001 L CNN
-F 3 "https://www.amphenolcanada.com/ProductSearch/drawings/AC/UE27ACX4X0X.pdf" H 6200 4850 60  0001 L CNN
-F 4 "UE27AC54100" H 6200 5050 60  0001 L CNN "MPN"
-F 5 "Amphenol ICC (Commercial Products)" H 6200 5650 60  0001 L CNN "Manufacturer"
-	1    6000 4550
-	1    0    0    -1
-$EndComp
-Wire Wire Line
-	6125 4875 6125 5050
-Wire Wire Line
-	6125 5050 6450 5050
-Wire Wire Line
-	6450 5050 6450 4650
+P 6000 4450
+F 0 "J5" H 6050 4850 60  0000 C CNN
+F 1 "UE27AC54100" H 5800 4100 60  0000 C CNN
+F 2 "antmicro-footprints:USB_A_Female_UE27AC54100" H 6200 4650 60  0001 L CNN
+F 3 "https://www.amphenolcanada.com/ProductSearch/drawings/AC/UE27ACX4X0X.pdf" H 6200 4750 60  0001 L CNN
+F 4 "UE27AC54100" H 6200 4950 60  0001 L CNN "MPN"
+F 5 "Amphenol ICC (Commercial Products)" H 6200 5550 60  0001 L CNN "Manufacturer"
+	1    6000 4450
+	1    0    0    1
+$EndComp
 Wire Wire Line
 	6450 4650 6300 4650
-Wire Wire Line
-	6450 5050 6450 5250
-Connection ~ 6450 5050
 $Comp
 L power:GND #PWR0109
@@
 Wire Wire Line
 	6650 5350 6650 5850
-Wire Wire Line
-	6650 5850 6750 5850
 Connection ~ 6650 5350
-$Comp
-L antmicro_Ferrite_Beads_and_Chips:BLM21PG221SN1D FB1
-U 1 1 5D853F7D
-P 6950 5850
-F 0 "FB1" H 6950 6137 60  0000 C CNN
-F 1 "BLM21PG221SN1D" H 6950 6031 60  0000 C CNN
-F 2 "antmicro-footprints:0805" H 7150 6050 60  0001 L CNN
-F 3 "https://www.murata.com/en-us/products/en-us/products/productdata/8796738977822/ENFA0005.pdf" H 7150 6150 60  0001 L CNN
-F 4 "BLM21PG221SN1D" H 7150 6350 60  0001 L CNN "MPN"
-F 5 "Murata Electronics North America" H 7150 6950 60  0001 L CNN "Manufacturer"
-	1    6950 5850
-	1    0    0    -1
-$EndComp
-Wire Wire Line
-	7150 5850 7250 5850
 Wire Wire Line
 	7800 5850 7800 5600
@@
 Wire Wire Line
 	5650 2300 5650 2200
-$Comp
-L antmicro_Resistors_0603:R_0R_0603 R11
-U 1 1 5DAF8709
-P 8800 4050
-F 0 "R11" V 8755 4120 60  0000 L CNN
-F 1 "R_0R_0603" H 8800 3900 60  0001 C CNN
-F 2 "antmicro-footprints:0603-res" H 9000 4250 60  0001 L CNN
-F 3 "" H 8800 4050 50  0001 C CNN
-F 4 "BOURNS" H 9000 4450 60  0001 L CNN "Manufacturer"
-F 5 "CR0603-J/-000ELF" H 9000 4350 60  0001 L CNN "MPN"
-F 6 "0R" V 8853 4120 50  0000 L CNN "Val"
-	1    8800 4050
-	0    1    1    0
-$EndComp
 Wire Wire Line
 	8800 3850 8800 3900
@@
 Connection ~ 7600 1850
 $Comp
-L antmicro_Capacitors_0402:C_100n_0402_6V3 C15
+L HDMI_SD_expansion-rescue:C_100n_0402_6V3-antmicro_Capacitors_0402 C15
 U 1 1 5DBC649D
 P 6950 3950
@@
 Wire Wire Line
 	6950 4200 6950 4100
-Text Notes 6000 6100 0    50   ~ 0
-Co to jest? Było w tym Reference od \nArduino i w bibliotece to wstawiłem.
 $Comp
 L antmicro_Test_Points:TP_SMD1MM TP1
@@
 	0    -1   -1   0
 $EndComp
-Text Notes 5400 3600 0    50   ~ 0
-Tutaj jeszcze bezpiecznik na 500mA \nale chyba musze go zrobic najpierw
-Text Notes 3550 5350 0    50   ~ 0
-Dodać ogranicznik prądu?
 Wire Wire Line
 	6000 2300 6000 2400
@@
 	1    0    0    -1
 $EndComp
+Text Notes 5000 2950 0    50   ~ 10
+caps will be replaced with 0R by default
+$Comp
+L antmicro_Resistors_0603:R_10k_0603 R11
+U 1 1 5D77F979
+P 8800 4050
+F 0 "R11" V 8755 4120 60  0000 L CNN
+F 1 "R_10k_0603" H 8800 3900 60  0001 C CNN
+F 2 "antmicro-footprints:0603-res" H 9000 4250 60  0001 L CNN
+F 3 "" H 8800 4050 50  0001 C CNN
+F 4 "BOURNS" H 9000 4450 60  0001 L CNN "Manufacturer"
+F 5 "CR0603-JW-103ELF" H 9000 4350 60  0001 L CNN "MPN"
+F 6 "10k" V 8853 4120 50  0000 L CNN "Val"
+	1    8800 4050
+	0    1    1    0
+$EndComp
+Wire Wire Line
+	6650 5850 7250 5850
+Text Label 1800 2400 0    50   ~ 0
+GPX_USB
+Text Label 1800 2500 0    50   ~ 0
+RST_USB
+Wire Wire Line
+	6450 4650 6450 5250
 $EndSCHEMATC

Commit message: Added testpads
Parts:
- added TP10, TP4, TP5, TP6, TP7, TP8, TP9: TP_SMD1MM, antmicro-footprints:Testpoint_smd_1mm, symbol antmicro_Test_Points:TP_SMD1MM
Connections:
- net GPX_USB: now also TP10.1
- net MISO_USB: now also TP8.1
- net MOSI_USB: now also TP9.1
- net RST_USB: now also TP5.1
- net SCK_USB: now also TP6.1
- net SS_USB: now also TP7.1
- net INT_USB: now reaches R11.2, U2.18 (INT)
- net INT_USB: now also J6.9, TP4.1
Other:
- moved on the sheet: J6
Changed lines of the file:
@@
 L antmicro_Rectangular_Connectors_Headers_Male_Pins:0015912120 J6
 U 1 1 5DC8649C
-P 1400 2600
-F 0 "J6" H 1400 3047 60  0000 C CNN
-F 1 "0015912120" H 1400 2941 60  0000 C CNN
-F 2 "antmicro-footprints:PinHeader_6x2_P2.54mm_Horizontal_Mirrored" H 1600 2800 60  0001 L CNN
-F 3 "https://www.molex.com/pdm_docs/sd/015912120_sd.pdf" H 1600 2900 60  0001 L CNN
-F 4 "0015912120" H 1600 3100 60  0001 L CNN "MPN"
-F 5 "Molex" H 1600 3700 60  0001 L CNN "Manufacturer"
-	1    1400 2600
+P 1600 2600
+F 0 "J6" H 1600 3047 60  0000 C CNN
+F 1 "0015912120" H 1600 2941 60  0000 C CNN
+F 2 "antmicro-footprints:PinHeader_6x2_P2.54mm_Horizontal_Mirrored" H 1800 2800 60  0001 L CNN
+F 3 "https://www.molex.com/pdm_docs/sd/015912120_sd.pdf" H 1800 2900 60  0001 L CNN
+F 4 "0015912120" H 1800 3100 60  0001 L CNN "MPN"
+F 5 "Molex" H 1800 3700 60  0001 L CNN "Manufacturer"
+	1    1600 2600
 	1    0    0    -1
 $EndComp
 Wire Wire Line
-	1200 2400 650  2400
+	1400 2400 850  2400
 Wire Wire Line
-	1200 2600 650  2600
-Text Label 650  2400 0    50   ~ 0
+	1400 2600 850  2600
+Text Label 850  2400 0    50   ~ 0
 SS_USB
-Text Label 650  2600 0    50   ~ 0
+Text Label 850  2600 0    50   ~ 0
 MISO_USB
 Wire Wire Line
-	2150 2400 1600 2400
+	2350 2400 1800 2400
 Wire Wire Line
-	1600 2500 2150 2500
+	1800 2500 2350 2500
 Wire Wire Line
-	1200 2500 650  2500
+	1400 2500 850  2500
 Wire Wire Line
-	1200 2700 650  2700
-Text Label 650  2500 0    50   ~ 0
+	1400 2700 850  2700
+Text Label 850  2500 0    50   ~ 0
 MOSI_USB
-Text Label 650  2700 0    50   ~ 0
+Text Label 850  2700 0    50   ~ 0
 SCK_USB
 Wire Wire Line
-	1600 2600 2150 2600
+	1800 2600 2350 2600
 Wire Wire Line
-	2150 2700 1600 2700
+	2350 2700 1800 2700
 Wire Wire Line
-	650  2800 1200 2800
-Text Label 650  2800 0    50   ~ 0
+	850  2800 1400 2800
+Text Label 850  2800 0    50   ~ 0
 GND
-Text Label 650  2900 0    50   ~ 0
+Text Label 850  2900 0    50   ~ 0
 +3V3
 Wire Wire Line
-	1200 2900 650  2900
+	1400 2900 850  2900
 Wire Wire Line
-	2150 2800 1600 2800
-Text Label 2150 2800 2    50   ~ 0
+	2350 2800 1800 2800
+Text Label 2350 2800 2    50   ~ 0
 GND
-Text Label 2150 2900 2    50   ~ 0
+Text Label 2350 2900 2    50   ~ 0
 +3V3
 Wire Wire Line
-	1600 2900 2150 2900
+	1800 2900 2350 2900
 Text Notes 600  2000 0    98   ~ 0
 USB_CON_#3
@@
 Wire Wire Line
 	6650 5850 7250 5850
-Text Label 1800 2400 0    50   ~ 0
+Text Label 2000 2400 0    50   ~ 0
 GPX_USB
-Text Label 1800 2500 0    50   ~ 0
+Text Label 2000 2500 0    50   ~ 0
 RST_USB
 Wire Wire Line
 	6450 4650 6450 5250
+Wire Wire Line
+	8800 4250 8200 4250
+Connection ~ 8800 4250
+Text Label 8200 4250 0    50   ~ 0
+INT_USB
+Text Label 2350 2600 2    50   ~ 0
+INT_USB
+$Comp
+L antmicro_Test_Points:TP_SMD1MM TP5
+U 1 1 5D79AD74
+P 8100 5050
+F 0 "TP5" V 8100 4950 50  0000 C CNN
+F 1 "TP_SMD1MM" H 8100 4950 50  0001 C CNN
+F 2 "antmicro-footprints:Testpoint_smd_1mm" H 8300 5250 60  0001 L CNN
+F 3 "" H 8300 5350 60  0001 L CNN
+	1    8100 5050
+	0    1    1    0
+$EndComp
+$Comp
+L antmicro_Test_Points:TP_SMD1MM TP6
+U 1 1 5D79AE8D
+P 8100 5150
+F 0 "TP6" V 8100 5050 50  0000 C CNN
+F 1 "TP_SMD1MM" H 8100 5050 50  0001 C CNN
+F 2 "antmicro-footprints:Testpoint_smd_1mm" H 8300 5350 60  0001 L CNN
+F 3 "" H 8300 5450 60  0001 L CNN
+	1    8100 5150
+	0    1    1    0
+$EndComp
+$Comp
+L antmicro_Test_Points:TP_SMD1MM TP7
+U 1 1 5D79AEFF
+P 8100 5250
+F 0 "TP7" V 8100 5150 50  0000 C CNN
+F 1 "TP_SMD1MM" H 8100 5150 50  0001 C CNN
+F 2 "antmicro-footprints:Testpoint_smd_1mm" H 8300 5450 60  0001 L CNN
+F 3 "" H 8300 5550 60  0001 L CNN
+	1    8100 5250
+	0    1    1    0
+$EndComp
+$Comp
+L antmicro_Test_Points:TP_SMD1MM TP8
+U 1 1 5D79AF73
+P 8100 5350
+F 0 "TP8" V 8100 5250 50  0000 C CNN
+F 1 "TP_SMD1MM" H 8100 5250 50  0001 C CNN
+F 2 "antmicro-footprints:Testpoint_smd_1mm" H 8300 5550 60  0001 L CNN
+F 3 "" H 8300 5650 60  0001 L CNN
+	1    8100 5350
+	0    1    1    0
+$EndComp
+$Comp
+L antmicro_Test_Points:TP_SMD1MM TP9
+U 1 1 5D79AFE9
+P 8100 5450
+F 0 "TP9" V 8100 5350 50  0000 C CNN
+F 1 "TP_SMD1MM" H 8100 5350 50  0001 C CNN
+F 2 "antmicro-footprints:Testpoint_smd_1mm" H 8300 5650 60  0001 L CNN
+F 3 "" H 8300 5750 60  0001 L CNN
+	1    8100 5450
+	0    1    1    0
+$EndComp
+$Comp
+L antmicro_Test_Points:TP_SMD1MM TP10
+U 1 1 5D79B061
+P 8100 5550
+F 0 "TP10" V 8100 5450 50  0000 C CNN
+F 1 "TP_SMD1MM" H 8100 5450 50  0001 C CNN
+F 2 "antmicro-footprints:Testpoint_smd_1mm" H 8300 5750 60  0001 L CNN
+F 3 "" H 8300 5850 60  0001 L CNN
+	1    8100 5550
+	0    1    1    0
+$EndComp
+$Comp
+L antmicro_Test_Points:TP_SMD1MM TP4
+U 1 1 5D79B146
+P 8100 4250
+F 0 "TP4" V 8100 4150 50  0000 C CNN
+F 1 "TP_SMD1MM" H 8100 4150 50  0001 C CNN
+F 2 "antmicro-footprints:Testpoint_smd_1mm" H 8300 4450 60  0001 L CNN
+F 3 "" H 8300 4550 60  0001 L CNN
+	1    8100 4250
+	0    1    1    0
+$EndComp
 $EndSCHEMATC
