File: Arty_HDMI_SD/_autosave-HDMI_SD_expansion.kicad_pcb (KiCad board)
At the start: 4 copper layers, 109 x 40 mm, 60 parts, among them IC1 TPD8S009DSMR, J2 1140084168, J4 2000-1-2-41-00-BK, J5 UE27AC54100, U1 TPS61232DRCT, U2 MAX3421EEHJ, Y1 KX-7_12,MHz

Commit message: Added TVS
Parts:
- added D3: TPD6E05U06, antmicro-footprints:TPD6E05U06, F.Cu at (176.7, 112.8)
- moved R2 15.2 mm to (182.5, 110.2)
- moved R7 14.7 mm to (180.8, 110.2)
- moved R4 4.52 mm to (179.2, 108.1)
- moved R3 4.24 mm to (177.3, 108.1)
- moved R5 4.06 mm to (175.5, 108.1)
- moved R6 4.00 mm to (173.7, 108.1)
- moved R1 3.59 mm to (189.0, 114.0)
- moved R12 1.91 mm to (190.3, 114.2)
- moved C1 0.36 mm to (186.1, 104.3)
Routing:
- net /DAT1: track 37.3 -> 59.6 mm
- net /DAT2: track 42.5 -> 62.8 mm
- net /MISO_DAT0: track 28.7 -> 40.3 mm
- net /SCK: track 26.4 -> 36.0 mm
- net GND: track 78.7 -> 86.5 mm, vias 31 -> 29
- net /MOSI_CMD: track 33.1 -> 38.9 mm
- net /CD_DAT3: track 36.5 -> 41.9 mm
- net +3V3: track 42.9 -> 39.9 mm
- net Net-(J2-Pad9): track 5.64 -> 3.68 mm
- net /CD: track 21.9 -> 21.6 mm, vias 0 -> 2
