File: Arty_HDMI_SD/_saved_HDMI_SD_expansion.sch (KiCad schematic (older format))
At the start: 60 parts, among them J2 1140084168, J4 2000-1-2-41-00-BK, J5 UE27AC54100, U1 TPS61232DRCT, U2 MAX3421EEHJ, Y1 KX-7_12,MHz

Commit message: Added TVS
Parts:
- added D3: TPD6E05U06, antmicro-footprints:TPD6E05U06, symbol antmicroTVSDiodes:TPD6E05U06
- gave numbers to parts that had none: 1
Connections:
- wire segments 270 -> 287
Other:
- moved on the sheet: R1, R12, R2, R3, R4, R5, R6, R7
