File: arty-a7-expansion.sch (KiCad schematic (older format))
At the start: 121 parts, among them IC1 TPD8S009DSMR, IC2 PCA9500PW, J1 SJ-43516-SMT-GR, J3 SJ-43516-SMT-BE, J4 685119134923, J5 UE27AC54100, U1 TPS61232DRCT, U2 MAX3421EEHJ, U3 CS4344-CZZ, U4 CS5343-CZZ, U5 NC7SZ126P5X, Y1 ABM8G-12.000MHZ-18-D2Y-T

Commit message: Add 5V0 led indicator
Parts:
- removed R44: R_100R_0402, arty-a7-expansion-footprints:0402-res, symbol arty-a7-expansion:R_100R_0402
- added D8: LG_L29K-G2J1-24-Z, arty-a7-expansion-footprints:LED_0603, symbol arty-a7-expansion:LG_L29K-G2J1-24-Z
- added Q1: BSS138APW, antmicro-footprints:SC70-3, symbol antmicroTransistorsFETsMOSFETsSingle:BSS138APW
- added R44, R46: R_330R_0402, antmicro-footprints:0402-res, symbol antmicroResistors0402:R_330R_0402
- added R45: R_10k_0402, antmicro-footprints:0402-res, symbol antmicroResistors0402:R_10k_0402
- gave numbers to parts that had none: 1
Connections:
- net +3V3: now also D8.1
- net GND: now also Q1.2 (S), R44.2
- net 5V0: now reaches C12.1, C13.1, C14.1, R8.2, TP3.1, U1.3 (VOUT), U1.4 (VOUT), U1.7 (FB)
- net 5V0: now also R45.2
- net 5V0_PG: now reaches TP2.1, U1.5 (PG)
- net 5V0_PG: now also Q1.1 (G), R45.1
- net at D7.2: now also R44.1
- new net: D8.2, R46.2
- new net: Q1.3 (D), R46.1
Changed lines of the file:
@@
 Connection ~ 2400 5600
-$Comp
-L arty-a7-expansion:R_100R_0402 R44
-U 1 1 5FDBB3B2
-P 6900 2200
-F 0 "R44" H 6900 2100 60  0000 C CNN
-F 1 "R_100R_0402" H 6900 2050 60  0001 C CNN
-F 2 "arty-a7-expansion-footprints:0402-res" H 7100 2400 60  0001 L CNN
-F 3 "" H 6900 2200 50  0001 C CNN
-F 4 "BOURNS" H 7100 2600 60  0001 L CNN "Manufacturer"
-F 5 "CR0402-FX-1000GLF" H 7100 2500 60  0001 L CNN "MPN"
-F 6 "100R" H 6900 2300 50  0000 C CNN "Val"
-	1    6900 2200
-	0    1    1    0
-$EndComp
 $Comp
 L arty-a7-expansion:LG_L29K-G2J1-24-Z D7
@@
 Wire Wire Line
 	6900 2350 6900 2400
-Text Notes 6350 1400 0    118  ~ 24
+Text Notes 7250 1100 0    118  ~ 24
 PWR indicator
 $Comp
-L arty-a7-expansion:DM3AT-SF-PEJM5 J?
+L arty-a7-expansion:DM3AT-SF-PEJM5 J2
 U 1 1 6112B8A7
 P 17550 11850
-F 0 "J?" H 17500 12849 50  0000 C CNN
+F 0 "J2" H 17500 12849 50  0000 C CNN
 F 1 "DM3AT-SF-PEJM5" H 17500 12758 50  0000 C CNN
 F 2 "arty-a7-expansion-footprints:MicroSD_DM3AT-SF-PEJM5" H 17550 11850 50  0001 C CNN
@@
 	1    0    0    -1
 $EndComp
+$Comp
+L arty-a7-expansion:LG_L29K-G2J1-24-Z D8
+U 1 1 601ED244
+P 9925 1900
+F 0 "D8" H 9900 1825 60  0000 L CNN
+F 1 "LG_L29K-G2J1-24-Z" H 9025 2100 60  0000 L CNN
+F 2 "arty-a7-expansion-footprints:LED_0603" H 10125 2100 60  0001 L CNN
+F 3 "https://dammedia.osram.info/media/resource/hires/osram-dam-2493945/LG%20L29K.pdf" H 10125 2200 60  0001 L CNN
+F 4 "LG L29K-G2J1-24-Z" H 10125 2400 60  0001 L CNN "MPN"
+F 5 "OSRAM Opto Semiconductors Inc." H 10125 3000 60  0001 L CNN "Manufacturer"
+	1    9925 1900
+	-1   0    0    1
+$EndComp
+Text Label 19400 11650 0    50   ~ 0
+5V0_PG
+Text Label 8125 2400 0    50   ~ 0
+5V0_PG
+$Comp
+L antmicroTransistorsFETsMOSFETsSingle:BSS138APW Q1
+U 1 1 601FEEC3
+P 9025 2300
+F 0 "Q1" H 9133 2353 60  0000 L CNN
+F 1 "BSS138APW" H 9133 2247 60  0000 L CNN
+F 2 "antmicro-footprints:SC70-3" H 9225 2500 60  0001 L CNN
+F 3 "" H 9225 2600 60  0001 L CNN
+F 4 "BSS138PW" H 9225 2800 60  0001 L CNN "MPN"
+F 5 "ON Semiconductor" H 9225 3400 60  0001 L CNN "Manufacturer"
+	1    9025 2300
+	1    0    0    -1
+$EndComp
+$Comp
+L arty-a7-expansion:+3V3 #PWR0143
+U 1 1 602088AF
+P 10350 1775
+F 0 "#PWR0143" H 10350 1625 50  0001 C CNN
+F 1 "+3V3" H 10365 1948 50  0000 C CNN
+F 2 "" H 10350 1775 50  0001 C CNN
+F 3 "" H 10350 1775 50  0001 C CNN
+	1    10350 1775
+	1    0    0    -1
+$EndComp
+Wire Wire Line
+	10350 1775 10350 1900
+Wire Wire Line
+	10350 1900 10125 1900
+Wire Wire Line
+	9375 1900 9025 1900
+Wire Wire Line
+	9025 1900 9025 2100
+Wire Wire Line
+	9025 2500 9025 2750
+$Comp
+L arty-a7-expansion:GND #PWR0144
+U 1 1 603065BA
+P 9025 2750
+F 0 "#PWR0144" H 9025 2500 50  0001 C CNN
+F 1 "GND" H 9030 2577 50  0000 C CNN
+F 2 "" H 9025 2750 50  0001 C CNN
+F 3 "" H 9025 2750 50  0001 C CNN
+	1    9025 2750
+	1    0    0    -1
+$EndComp
+Wire Wire Line
+	8725 2400 8650 2400
+Connection ~ 8650 2400
+Wire Wire Line
+	8650 2400 8125 2400
+$Comp
+L antmicroResistors0402:R_10k_0402 R45
+U 1 1 603D1739
+P 8425 2050
+F 0 "R45" H 8375 1950 60  0000 L CNN
+F 1 "R_10k_0402" H 8425 1900 60  0001 C CNN
+F 2 "antmicro-footprints:0402-res" H 8625 2250 60  0001 L CNN
+F 3 "" H 8425 2050 50  0001 C CNN
+F 4 "VISHAY" H 8625 2450 60  0001 L CNN "Manufacturer"
+F 5 "CRCW040210K0FKEDHP" H 8625 2350 60  0001 L CNN "MPN"
+F 6 "10k" H 8375 2150 50  0000 L CNN "Val"
+	1    8425 2050
+	-1   0    0    1
+$EndComp
+Wire Wire Line
+	8275 2050 8125 2050
+$Comp
+L antmicroResistors0402:R_330R_0402 R44
+U 1 1 60477F03
+P 6900 2200
+F 0 "R44" V 6855 2270 60  0000 L CNN
+F 1 "R_330R_0402" H 6900 2050 60  0001 C CNN
+F 2 "antmicro-footprints:0402-res" H 7100 2400 60  0001 L CNN
+F 3 "" H 6900 2200 50  0001 C CNN
+F 4 "MULTICOMP" H 7100 2600 60  0001 L CNN "Manufacturer"
+F 5 "MCMR04X3300FTL" H 7100 2500 60  0001 L CNN "MPN"
+F 6 "330R" V 6953 2270 50  0000 L CNN "Val"
+	1    6900 2200
+	0    1    1    0
+$EndComp
+Wire Wire Line
+	9825 1900 9675 1900
+$Comp
+L antmicroResistors0402:R_330R_0402 R46
+U 1 1 604774DC
+P 9525 1900
+F 0 "R46" H 9325 1975 60  0000 C CNN
+F 1 "R_330R_0402" H 9525 1750 60  0001 C CNN
+F 2 "antmicro-footprints:0402-res" H 9725 2100 60  0001 L CNN
+F 3 "" H 9525 1900 50  0001 C CNN
+F 4 "MULTICOMP" H 9725 2300 60  0001 L CNN "Manufacturer"
+F 5 "MCMR04X3300FTL" H 9725 2200 60  0001 L CNN "MPN"
+F 6 "330R" H 9525 1800 50  0000 C CNN "Val"
+	1    9525 1900
+	1    0    0    -1
+$EndComp
+Text Label 21425 11450 0    50   ~ 0
+5V0
+Text Label 8125 2050 0    50   ~ 0
+5V0
+Wire Wire Line
+	8650 2050 8575 2050
+Wire Wire Line
+	8650 2050 8650 2400
 $EndSCHEMATC
